Commit message: Gantry robot is working in Gazebo.

File: kh_sandbox/urdf/arm.transmission.xacro (robot description, xacro)
@@ -5,4 +5,14 @@
        xmlns:xacro="http://ros.org/wiki/xacro">
 	<xacro:macro name="ur_arm_transmission" params="name">
+		<transmission name="gantry_xbar_trans" type="pr2_mechanism_model/SimpleTransmission">
+			<actuator name="gantry_xbar_motor"/>
+			<joint name="gantry_xbar_joint"/>
+			<mechanicalReduction>1</mechanicalReduction>
+		</transmission>
+		<transmission name="gantry_center_trans" type="pr2_mechanism_model/SimpleTransmission">
+			<actuator name="gantry_center_motor"/>
+			<joint name="gantry_center_joint"/>
+			<mechanicalReduction>1</mechanicalReduction>
+		</transmission>
 		<transmission name="shoulder_pan_trans" type="pr2_mechanism_model/SimpleTransmission">
 			<actuator name="shoulder_pan_motor"/>

File: kh_sandbox/urdf/model.urdf.xacro (robot description, xacro)
@@ -50,13 +50,55 @@
   <property name="elbow_collision_length" value="0.200" />     <!-- manually measured -->
   <property name="elbow_collision_offset" value="0.035" />     <!-- manually measured -->
+<!-- Gantry model -->
+  <property name="gantry_height" value="2.43" />
   <link name="base_link" >
-  </link>
+    <inertial>
+      <mass value="15" />
+      <inertia ixx="1.0" ixy="0.0" ixz="0.0" iyy="1.0" iyz="0.0" izz="1.0"/>
+    </inertial>
+  </link>
+<xacro:macro name="gantry_leg" params="leg_name leg_x leg_y">
+  <link name="gantry_leg_${leg_name}">
+    <visual>
+      <geometry>
+          <box size="0.1 0.1 ${gantry_height}" />
+      </geometry>
+      <material name="orange">
+        <color rgba="1 .6 0 1" />
+      </material>
+    </visual>
+    <collision>
+      <geometry>
+          <box size="0.1 0.1 ${gantry_height}" />
+      </geometry>
+    </collision>
+    <inertial>
+      <mass value="1000" />
+      <inertia ixx="1.0" ixy="0.0" ixz="0.0" iyy="1.0" iyz="0.0" izz="1.0"/>
+      <origin xyz="0.0 0.0 0.0" rpy="0.0 0.0 0.0" />
+    </inertial>
+  </link>
+  <joint name="gantry_leg_${leg_name}_joint" type="fixed">
+    <parent link = "gantry_frame_link" />
+    <child link="gantry_leg_${leg_name}" />
+    <origin xyz="${leg_x} ${leg_y} ${-gantry_height}" rpy="0.0 0.0 0.0" />
+    <axis xyz="0.0 0.0 1.0" />
+  </joint>
+</xacro:macro>
+<xacro:gantry_leg leg_name="1" leg_x="${1.5/2.0}" leg_y="${1.5/2.0}" />
+<xacro:gantry_leg leg_name="2" leg_x="${-1.5/2.0}" leg_y="${1.5/2.0}" />
+<xacro:gantry_leg leg_name="3" leg_x="${-1.5/2.0}" leg_y="${-1.5/2.0}" />
+<xacro:gantry_leg leg_name="4" leg_x="${1.5/2.0}" leg_y="${-1.5/2.0}" />
   <joint name="gantry_frame_joint" type="fixed">
     <parent link = "base_link" />
     <child link="gantry_frame_link" />
-    <origin xyz="0.0 0.0 2.43" rpy="0.0 0.0 0.0" />
+    <origin xyz="0.0 0.0 ${gantry_height}" rpy="0.0 0.0 0.0" />
     <axis xyz="0.0 0.0 1.0" />
   </joint>
   <link name="gantry_frame_link" >
+    <inertial>
+      <mass value="15" />
+      <inertia ixx="1.0" ixy="0.0" ixz="0.0" iyy="1.0" iyz="0.0" izz="1.0"/>
+    </inertial>
   </link>
   <joint name="gantry_xbar_joint" type="prismatic">
@@ -68,4 +110,8 @@
   </joint>
   <link name="gantry_xbar_link" >
+    <inertial>
+      <mass value="15" />
+      <inertia ixx="1.0" ixy="0.0" ixz="0.0" iyy="1.0" iyz="0.0" izz="1.0"/>
+    </inertial>
   </link>
   <joint name="gantry_center_joint" type="prismatic">
@@ -77,4 +123,8 @@
   </joint>
   <link name="gantry_center_link" >
+    <inertial>
+      <mass value="15" />
+      <inertia ixx="1.0" ixy="0.0" ixz="0.0" iyy="1.0" iyz="0.0" izz="1.0"/>
+    </inertial>
   </link>
   <joint name="gantry_mount_joint" type="fixed">
@@ -85,4 +135,8 @@
   </joint>
   <link name="gantry_mount_link" >
+    <inertial>
+      <mass value="1" />
+      <inertia ixx="1.0" ixy="0.0" ixz="0.0" iyy="1.0" iyz="0.0" izz="1.0"/>
+    </inertial>
   </link>
 <xacro:macro name="ur5_robot" params="arm_name">
