Commit message: Old stuff from imkr control tests.

File: kh_sandbox/urdf/model.urdf.xacro (robot description, xacro)
@@ -74,5 +74,5 @@
     </collision>
     <inertial>
-      <mass value="1000" />
+      <mass value="100" />
       <inertia ixx="1.0" ixy="0.0" ixz="0.0" iyy="1.0" iyz="0.0" izz="1.0"/>
       <origin xyz="0.0 0.0 0.0" rpy="0.0 0.0 0.0" />
@@ -82,5 +82,5 @@
     <parent link = "gantry_frame_link" />
     <child link="gantry_leg_${leg_name}" />
-    <origin xyz="${leg_x} ${leg_y} ${-gantry_height}" rpy="0.0 0.0 0.0" />
+    <origin xyz="${leg_x} ${leg_y} ${-gantry_height/2}" rpy="0.0 0.0 0.0" />
     <axis xyz="0.0 0.0 1.0" />
   </joint>
