Commit message: Added cart base to URDF/collada model, added notes on how to make new collada files.

File: universal_robot_cpl/ur10_description/ur10_robot.urdf (robot description, URDF)
Before this commit: robot ur10, 9 links, 8 joints
Links:
- added link cart_base_link, mass 100; collision box size=1.22 0.62 0.915; visual mesh filename=package://ur10_description/meshes/cube.dae scale=1.22 0.62 0.915
- added link forearm_middle_link, mass 0; collision cylinder length=0.45 radius=0.043
- added link upper_arm_middle_link, mass 0; collision cylinder length=0.45 radius=0.0525
- link forearm_link: geometry collision cylinder length=0.26 radius=0.06; visual mesh filename=package://ur10_description/meshes/Forearm.dae scale=0.001 0.001 0.001
- link upper_arm_link: geometry visual mesh filename=package://ur10_description/meshes/UpperArm.dae scale=0.001 0.001 0.001
- link upper_shoulder_link: geometry collision cylinder length=0.175 radius=0.075
- link wrist_1_link: geometry collision cylinder length=0.123 radius=0.045; visual mesh filename=package://ur10_description/meshes/Wrist1.dae scale=0.001 0.001 0.001
- link wrist_2_link: geometry collision cylinder length=0.123 radius=0.045; visual mesh filename=package://ur10_description/meshes/Wrist2.dae scale=0.001 0.001 0.001
- link wrist_3_link: geometry collision cylinder length=0.148 radius=0.045; visual mesh filename=package://ur10_description/meshes/Wrist3.dae scale=0.001 0.001 0.001
Joints:
- added joint cart_base_joint: type fixed, parent base_link, child cart_base_link, origin xyz=0.08 -0.12 -0.915 rpy=0.0 0.0 0.0
- added joint forearm_middle_joint: type fixed, parent forearm_link, child forearm_middle_link, origin xyz=0.0 0.0 0.295 rpy=0.0 0.0 0.0
- added joint upper_arm_middle_joint: type fixed, parent upper_arm_link, child upper_arm_middle_link, origin xyz=0.0 -0.046 0.32 rpy=-1.570796325 3.14159265 0.0
- joint upper_shoulder_joint: origin xyz=0.0 -0.053 0.0 rpy=-1.570796325 0.0 0.0 -> xyz=0.0 -0.046 0.0 rpy=-1.570796325 3.14159265 0.0

File: universal_robot_cpl/ur10_description/urdf/model.urdf.xacro (robot description, xacro)
@@ -54,5 +54,5 @@
   <property name="upper_arm_radius" value="0.054" />  <!-- manually measured -->
   <property name="elbow_radius" value="0.060" />      <!-- manually measured -->
-  <property name="forearm_radius" value="0.040" />    <!-- manually measured -->
+  <property name="forearm_radius" value="0.043" />    <!-- manually measured -->
   <property name="wrist_radius" value="0.045" />      <!-- manually measured -->
 <!-- Collision model -->
@@ -75,4 +75,68 @@
     </inertial>
   </link>
+  <joint name="${prefix}cart_base_joint" type="fixed">
+    <parent link="${prefix}base_link" />
+    <child link = "${prefix}cart_base_link" />
+    <origin xyz="0.08 -0.12 -0.915" rpy="0.0 0.0 0.0" />
+  </joint>
+  <link name="${prefix}cart_base_link">
+    <visual>
+      <!--
+      <geometry>
+          <box size="1.22 0.62 0.915" />
+      </geometry>
+      -->
+      <geometry>
+        <mesh filename="package://ur10_description/meshes/cube.dae" scale="1.22 0.62 0.915"/>
+      </geometry>
+      <origin xyz="-0.61 0.31 0.458" rpy="0.0 0.0 0.0" />
+      <material name="grey">
+          <color rgba="0.3 0.3 0.3 1" />
+      </material>
+    </visual>
+    <collision>
+      <geometry>
+          <box size="1.22 0.62 0.915" />
+      </geometry>
+      <origin xyz="-0.61 0.31 -0.458" rpy="0.0 0.0 0.0" />
+    </collision>
+    <inertial>
+      <mass value="100" />
+      <inertia ixx="1.0" ixy="0.0" ixz="0.0" iyy="1.0" iyz="0.0" izz="1.0"/>
+      <origin xyz="-0.61 0.31 -0.458" rpy="0.0 0.0 0.0" />
+    </inertial>
+  </link>
+  <joint name="${prefix}work_table_joint" type="fixed">
+    <parent link="${prefix}cart_base_link" />
+    <child link = "${prefix}work_table_link" />
+    <origin xyz="0.0 0.0 0.715" rpy="0.0 0.0 ${-3.0*pi/4.0}" />
+  </joint>
+  <link name="${prefix}work_table_link">
+      <!--
+    <visual>
+      <geometry>
+          <box size="1.22 0.62 0.915" />
+      </geometry>
+      <geometry>
+        <mesh filename="package://ur10_description/meshes/cube.dae" scale="1.22 0.62 0.915"/>
+      </geometry>
+      <origin xyz="-0.61 0.31 0.458" rpy="0.0 0.0 0.0" />
+      <material name="grey">
+          <color rgba="0.3 0.3 0.3 1" />
+      </material>
+    </visual>
+    <collision>
+      <geometry>
+          <box size="1.22 0.62 0.915" />
+      </geometry>
+      <origin xyz="-0.61 0.31 -0.458" rpy="0.0 0.0 0.0" />
+    </collision>
+      -->
+    <inertial>
+      <mass value="100" />
+      <inertia ixx="1.0" ixy="0.0" ixz="0.0" iyy="1.0" iyz="0.0" izz="1.0"/>
+      <origin xyz="-0.61 0.31 -0.458" rpy="0.0 0.0 0.0" />
+    </inertial>
+  </link>
   <joint name="${prefix}shoulder_pan_joint" type="revolute">
     <parent link="${prefix}base_link" />
@@ -110,15 +174,28 @@
     <dynamics damping="10" friction="0.1"/>
   </joint>
+  <link name="${prefix}upper_arm_link">
+    <visual>
+      <geometry>
+        <mesh filename="package://ur10_description/meshes/UpperArm.dae" scale="0.001 0.001 0.001"/>
+      </geometry>
+      <origin xyz="0.0 -0.221 -0.127" rpy="${pi / 2.0} -${0*pi / 2.0} 0.0" />
+    </visual>
+    <inertial>
+      <mass value="${upper_arm_mass}" />
+      <inertia ixx="1.0" ixy="0.0" ixz="0.0" iyy="1.0" iyz="0.0" izz="1.0"/>
+      <origin xyz="${upper_arm_cog}" rpy="0.0 0.0 0.0" />
+    </inertial>
+  </link>
   <joint name="${prefix}upper_shoulder_joint" type="fixed">
     <parent link="${prefix}upper_arm_link" />
     <child link = "${prefix}upper_shoulder_link" />
-    <origin xyz="0.0 -0.053 0.0" rpy="${-pi/2.0} 0.0 0.0" />
+    <origin xyz="0.0 -0.046 0.0" rpy="${-pi/2.0} ${pi} 0.0" />
   </joint>
   <link name="${prefix}upper_shoulder_link">
     <collision>
       <geometry>
-        <cylinder length="${base_collision_length}" radius="${shoulder_radius}"/>
-      </geometry>
-      <origin xyz="0.0 0.0 ${shoulder_height}" rpy="0.0 0.0 0.0" />
+        <cylinder length="0.175" radius="${shoulder_radius}"/>
+      </geometry>
+      <origin xyz="0.0 0.0 ${-(0.085-0.175/2.0)}" rpy="0.0 0.0 0.0" />
     </collision>
     <inertial>
@@ -128,21 +205,20 @@
     </inertial>
   </link>
-  <link name="${prefix}upper_arm_link">
-    <visual>
-      <geometry>
-        <mesh filename="package://ur10_description/meshes/UpperArm.dae" scale="0.001 0.001 0.001"/>
-      </geometry>
-      <origin xyz="0.0 -0.221 -0.127" rpy="${pi / 2.0} -${0*pi / 2.0} 0.0" />
-    </visual>
-    <collision>
-      <geometry>
-        <cylinder length="${upper_arm_length}" radius="${upper_arm_radius}"/>
-      </geometry>
-      <origin xyz="0.0 0.0 ${upper_arm_length/2.0}" rpy="0.0 0.0 0.0" />
-    </collision>
-    <inertial>
-      <mass value="${upper_arm_mass}" />
-      <inertia ixx="1.0" ixy="0.0" ixz="0.0" iyy="1.0" iyz="0.0" izz="1.0"/>
-      <origin xyz="${upper_arm_cog}" rpy="0.0 0.0 0.0" />
+  <joint name="${prefix}upper_arm_middle_joint" type="fixed">
+    <parent link="${prefix}upper_arm_link" />
+    <child link = "${prefix}upper_arm_middle_link" />
+    <origin xyz="0.0 -0.046 ${0.45/2.0+0.17-shoulder_radius}" rpy="${-pi/2.0} ${pi} 0.0" />
+  </joint>
+  <link name="${prefix}upper_arm_middle_link">
+    <collision>
+      <geometry>
+          <cylinder length="0.45" radius="${0.105/2.0}"/>
+      </geometry>
+      <origin xyz="0.0 0.0 0.0" rpy="${pi/2.0} 0.0 0.0" />
+    </collision>
+    <inertial>
+      <mass value="0" />
+      <inertia ixx="1.0" ixy="0.0" ixz="0.0" iyy="1.0" iyz="0.0" izz="1.0"/>
+      <origin xyz="0.0 0.0 0.0" rpy="0.0 0.0 0.0" />
     </inertial>
   </link>
@@ -164,7 +240,7 @@
     <collision>
       <geometry>
-        <cylinder length="${forearm_length}" radius="${forearm_radius}"/>
-      </geometry>
-      <origin xyz="0.0 0.0 ${forearm_length/2.0}" rpy="0.0 0.0 0.0" />
+          <cylinder length="0.26" radius="${0.12/2.0}"/>
+      </geometry>
+      <origin xyz="0.0 ${0.26/2.0-0.065} 0.0" rpy="${pi/2.0} 0.0 0.0" />
     </collision>
     <inertial>
@@ -172,4 +248,22 @@
       <origin xyz="${forearm_cog}" rpy="0.0 0.0 0.0" />
       <inertia ixx="1.0" ixy="0.0" ixz="0.0" iyy="1.0" iyz="0.0" izz="1.0"/>
+    </inertial>
+  </link>
+  <joint name="${prefix}forearm_middle_joint" type="fixed">
+    <parent link="${prefix}forearm_link" />
+    <child link = "${prefix}forearm_middle_link" />
+    <origin xyz="0.0 0.0 ${0.57-0.45/2.0-0.12/2.0+0.01}" rpy="0.0 0.0 0.0" />
+  </joint>
+  <link name="${prefix}forearm_middle_link">
+    <collision>
+      <geometry>
+          <cylinder length="0.45" radius="${forearm_radius}"/>
+      </geometry>
+      <origin xyz="0.0 0.0 0.0" rpy="0.0 0.0 0.0" />
+    </collision>
+    <inertial>
+      <mass value="0" />
+      <inertia ixx="1.0" ixy="0.0" ixz="0.0" iyy="1.0" iyz="0.0" izz="1.0"/>
+      <origin xyz="0.0 0.0 0.0" rpy="0.0 0.0 0.0" />
     </inertial>
   </link>
@@ -191,7 +285,7 @@
     <collision>
       <geometry>
-        <cylinder length="${1.6*wrist_1_length}" radius="${wrist_radius}"/>
-      </geometry>
-      <origin xyz="0.0 ${0.25*wrist_1_length} 0.0" rpy="${-pi/2.0} 0.0 0.0" />
+        <cylinder length="${0.123}" radius="${wrist_radius}"/>
+      </geometry>
+      <origin xyz="0.0 ${0.123/2.0-0.057} 0.0" rpy="${-pi/2.0} 0.0 0.0" />
     </collision>
     <inertial>
@@ -218,7 +312,7 @@
     <collision>
       <geometry>
-        <cylinder length="${1.6*wrist_2_length}" radius="${wrist_radius}"/>
-      </geometry>
-      <origin xyz="0.0 0.0 ${0.25*wrist_2_length}" rpy="0.0 0.0 0.0" />
+        <cylinder length="0.123" radius="${wrist_radius}"/>
+      </geometry>
+      <origin xyz="0.0 0.0 ${0.123/2.0-0.057}" rpy="0.0 0.0 0.0" />
     </collision>
     <inertial>
@@ -245,7 +339,7 @@
     <collision>
       <geometry>
-        <cylinder length="${1.65*wrist_3_length}" radius="${wrist_radius}"/>
-      </geometry>
-      <origin xyz="0.0 ${0.15 * wrist_3_length} 0.0" rpy="${-pi/2.0} 0.0 0.0" />
+          <cylinder length="${0.123+0.025}" radius="${wrist_radius}"/>
+      </geometry>
+      <origin xyz="0.0 ${(0.123+0.025)/2.0-0.057} 0.0" rpy="${-pi/2.0} 0.0 0.0" />
     </collision>
     <inertial>
