Commit message: Fixed URDF model.

File: universal_robot_cpl/ur10_description/urdf/model.urdf.xacro (robot description, xacro)
@@ -35,6 +35,6 @@
   <property name="wrist_3_mass" value="0.202" />
   <!-- TODO -->
-  <property name="shoulder_cog" value="0.0 0.00193 -0.02561" />
-  <property name="upper_arm_cog" value="0.0 -0.024201 0.2125" />   <!-- 0.11336 - 0.089159 =  -->
+  <property name="shoulder_cog" value="0.00008 0.00244 -0.037" />
+  <property name="upper_arm_cog" value="0.00008 0.00244   0.38757" />   <!-- 0.11336 - 0.089159 =  -->
   <property name="forearm_cog" value="0.0 0.0265 0.11993" />       <!-- 0.119 is not half of 0.39225, is this really correct? -->
   <property name="wrist_1_cog" value="0.0 0.110949 0.01634" />     <!-- 0.0018 + 0.10915 = 0.110949 -->
@@ -44,10 +44,10 @@
 <!-- Kinematic model -->
   <property name="shoulder_height" value="0.1273" />
-  <property name="shoulder_offset" value="0.13585" />  <!-- shoulder_offset - elbow_offset + wrist_1_length = 0.10915 -->
+  <property name="shoulder_offset" value="0.220941" />  <!-- shoulder_offset - elbow_offset + wrist_1_length = 0.220941 -->
   <property name="upper_arm_length" value="0.612" />
-  <property name="elbow_offset" value="0.1197" />       <!-- CAD measured TODO -->
+  <property name="elbow_offset" value="0.1719" />       <!-- CAD measured TODO -->
   <property name="forearm_length" value="0.5723" />
-  <property name="wrist_1_length" value="0.093" />     <!-- CAD measured TODO -->
-  <property name="wrist_2_length" value="0.1157" />   <!-- In CAD this distance is 0.930, but in the spec it is 0.09465 -->
+  <property name="wrist_1_length" value="0.1149" />     <!-- CAD measured TODO -->
+  <property name="wrist_2_length" value="0.1157" />
   <property name="wrist_3_length" value="0.0922" />
   <property name="shoulder_radius" value="0.075" />   <!-- manually measured -->
@@ -133,5 +133,5 @@
         <mesh filename="package://ur10_description/meshes/UpperArm.dae" scale="0.001 0.001 0.001"/>
       </geometry>
-      <origin xyz="0.0 -0.136 -0.127" rpy="${pi / 2.0} -${0*pi / 2.0} 0.0" />
+      <origin xyz="0.0 -0.221 -0.127" rpy="${pi / 2.0} -${0*pi / 2.0} 0.0" />
     </visual>
     <collision>
@@ -160,5 +160,5 @@
         <mesh filename="package://ur10_description/meshes/Forearm.dae" scale="0.001 0.001 0.001"/>
       </geometry>
-      <origin xyz="0.0 -0.016 -0.739" rpy="${pi / 2.0} 0.0 0.0" />
+      <origin xyz="0.0 -0.049 -0.739" rpy="${pi / 2.0} 0.0 0.0" />
     </visual>
     <collision>
@@ -187,5 +187,5 @@
         <mesh filename="package://ur10_description/meshes/Wrist1.dae" scale="0.001 0.001 0.001"/>
       </geometry>
-      <origin xyz="0.0 -0.016 -1.312" rpy="${pi / 2.0} 0.0 0.0" />
+      <origin xyz="0.0 -0.049 -1.312" rpy="${pi / 2.0} 0.0 0.0" />
     </visual>
     <collision>
@@ -214,5 +214,5 @@
         <mesh filename="package://ur10_description/meshes/Wrist2.dae" scale="0.001 0.001 0.001"/>
       </geometry>
-      <origin xyz="0.0 -0.109 -1.312" rpy="${pi / 2.0} 0.0 0.0" />
+      <origin xyz="0.0 -0.164 -1.312" rpy="${pi / 2.0} 0.0 0.0" />
     </visual>
     <collision>
@@ -241,5 +241,5 @@
         <mesh filename="package://ur10_description/meshes/Wrist3.dae" scale="0.001 0.001 0.001"/>
       </geometry>
-      <origin xyz="0.0 -0.109 -1.427" rpy="${pi / 2.0} 0.0 0.0" />
+      <origin xyz="0.0 -0.164 -1.427" rpy="${pi / 2.0} 0.0 0.0" />
     </visual>
     <collision>

Commit message: Updated robot description. Separated into robot's model and manipulation setup's model.

File: universal_robot_cpl/ur10_description/urdf/model.urdf.xacro (robot description, xacro)
@@ -75,68 +75,4 @@
     </inertial>
   </link>
-  <joint name="${prefix}cart_base_joint" type="fixed">
-    <parent link="${prefix}base_link" />
-    <child link = "${prefix}cart_base_link" />
-    <origin xyz="0.08 -0.12 -0.915" rpy="0.0 0.0 0.0" />
-  </joint>
-  <link name="${prefix}cart_base_link">
-    <visual>
-      <!--
-      <geometry>
-          <box size="1.22 0.62 0.915" />
-      </geometry>
-      -->
-      <geometry>
-        <mesh filename="package://ur10_description/meshes/cube.dae" scale="1.22 0.62 0.915"/>
-      </geometry>
-      <origin xyz="-0.61 0.31 0.458" rpy="0.0 0.0 0.0" />
-      <material name="grey">
-          <color rgba="0.3 0.3 0.3 1" />
-      </material>
-    </visual>
-    <collision>
-      <geometry>
-          <box size="1.22 0.62 0.915" />
-      </geometry>
-      <origin xyz="-0.61 0.31 -0.458" rpy="0.0 0.0 0.0" />
-    </collision>
-    <inertial>
-      <mass value="100" />
-      <inertia ixx="1.0" ixy="0.0" ixz="0.0" iyy="1.0" iyz="0.0" izz="1.0"/>
-      <origin xyz="-0.61 0.31 -0.458" rpy="0.0 0.0 0.0" />
-    </inertial>
-  </link>
-  <joint name="${prefix}work_table_joint" type="fixed">
-    <parent link="${prefix}cart_base_link" />
-    <child link = "${prefix}work_table_link" />
-    <origin xyz="0.0 0.0 0.715" rpy="0.0 0.0 ${-3.0*pi/4.0}" />
-  </joint>
-  <link name="${prefix}work_table_link">
-      <!--
-    <visual>
-      <geometry>
-          <box size="1.22 0.62 0.915" />
-      </geometry>
-      <geometry>
-        <mesh filename="package://ur10_description/meshes/cube.dae" scale="1.22 0.62 0.915"/>
-      </geometry>
-      <origin xyz="-0.61 0.31 0.458" rpy="0.0 0.0 0.0" />
-      <material name="grey">
-          <color rgba="0.3 0.3 0.3 1" />
-      </material>
-    </visual>
-    <collision>
-      <geometry>
-          <box size="1.22 0.62 0.915" />
-      </geometry>
-      <origin xyz="-0.61 0.31 -0.458" rpy="0.0 0.0 0.0" />
-    </collision>
-      -->
-    <inertial>
-      <mass value="100" />
-      <inertia ixx="1.0" ixy="0.0" ixz="0.0" iyy="1.0" iyz="0.0" izz="1.0"/>
-      <origin xyz="-0.61 0.31 -0.458" rpy="0.0 0.0 0.0" />
-    </inertial>
-  </link>
   <joint name="${prefix}shoulder_pan_joint" type="revolute">
     <parent link="${prefix}base_link" />
