Commit message: Centralizing the sensor/robot setup into URDF files

File: cpl_collab_manip/urdf/sensors.urdf.xacro (robot description, xacro)
@@ -4,18 +4,48 @@
        xmlns:interface="http://playerstage.sourceforge.net/gazebo/xmlschema/#interface"
        xmlns:xacro="http://ros.org/wiki/xacro">
+<property name="pi" value="3.14159265" />
 <xacro:macro name="sensors" params="prefix">
-  <property name="pi" value="3.14159265" />
   <joint name="${prefix}lifecam_joint" type="fixed">
     <parent link="${prefix}base_link" />
-    <child link = "${prefix}lifecam1_optical_frame" />
+    <child link = "lifecam1_optical_frame" />
     <origin xyz="0.260675 0.037183 1.903672" rpy="-2.78084434849 -0.0267970865698 1.96534931804" />
   </joint>
-  <link name="${prefix}lifecam1_optical_frame">
-    <inertial>
-      <mass value="100" />
-      <inertia ixx="1.0" ixy="0.0" ixz="0.0" iyy="1.0" iyz="0.0" izz="1.0"/>
-      <origin xyz="0.0 0.0 0.0" rpy="0.0 0.0 0.0" />
-    </inertial>
-  </link>
+  <link name="lifecam1_optical_frame"></link>
+  <joint name="${prefix}kinect0_calibration_joint" type="fixed">
+    <parent link="${prefix}base_link" />
+    <child link = "kinect0_calibration_frame" />
+    <origin xyz="0.433613 -0.406085 1.375427" rpy="-2.2212883 0.013399270 2.00038349" />
+  </joint>
+  <link name="kinect0_calibration_frame"></link>
+  <joint name="kinect0_base_joint" type="fixed">
+    <parent link="kinect0_calibration_frame" />
+    <child link = "kinect0_link" />
+    <origin xyz="-0.045 0.0 0.0" rpy="${pi / 2.0} -${pi / 2.0} 0.0" />
+  </joint>
+  <link name="kinect0_link"></link>
+  <joint name="kinect0_depth_joint" type="fixed">
+    <parent link="kinect0_link" />
+    <child link = "kinect0_depth_frame" />
+    <origin xyz="0.0 -0.02 0.0" rpy="0.0 0.0 0.0" />
+  </joint>
+  <link name="kinect0_depth_frame"></link>
+  <joint name="kinect0_rgb_joint" type="fixed">
+    <parent link="kinect0_link" />
+    <child link = "kinect0_rgb_frame" />
+    <origin xyz="0.0 -0.045 0.0" rpy="0.0 0.0 0.0" />
+  </joint>
+  <link name="kinect0_rgb_frame"></link>
+  <joint name="kinect0_depth_optical_joint" type="fixed">
+    <parent link="kinect0_depth_frame" />
+    <child link = "kinect0_depth_optical_frame" />
+    <origin xyz="0.0 0.0 0.0" rpy="-${pi/2.0} 0.0 -${pi/2.0}" />
+  </joint>
+  <link name="kinect0_depth_optical_frame"></link>
+  <joint name="kinect0_rgb_optical_joint" type="fixed">
+    <parent link="kinect0_rgb_frame" />
+    <child link = "kinect0_rgb_optical_frame" />
+    <origin xyz="0.0 0.0 0.0" rpy="-${pi/2.0} 0.0 -${pi/2.0}" />
+  </joint>
+  <link name="kinect0_rgb_optical_frame"></link>
 </xacro:macro>
 </robot>
